File: schematics/bootloadHID_sch.sch (EAGLE design)
At the start: 15 parts, among them IC1 MEGA8-P, J1 USB-B, Q1 12MHz, X1 J1

Commit message: Add files via upload
Parts:
- C3: value (none) -> 100uF
Changed lines of the file:
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@@
 <part name="X1" library="con-molex" deviceset="22-23-2021" device="" value="J1"/>
 <part name="J1" library="SparkFun-Connectors" deviceset="USB" device="PTH" value="USB-B"/>
-<part name="C3" library="adafruit" deviceset="CPOL-US" device="E2.5-6"/>
+<part name="C3" library="adafruit" deviceset="CPOL-US" device="E2.5-6" value="100uF"/>
 <part name="P+1" library="supply1" deviceset="VCC" device=""/>
 <part name="GND1" library="supply1" deviceset="GND" device=""/>
